File: main/pcb_challenge_final.kicad_pcb (KiCad board)
At the start: 4 copper layers, 66.2 x 38.8 mm, 164 parts, among them J4 Conn_01x04_Pin, J5 Conn_01x04_Pin, Q15 Q_Dual_NPN_PNP_B1E2B2C2E1C1, Q16 Q_Dual_NPN_PNP_B1E2B2C2E1C1, Q17 Q_Dual_NPN_PNP_B1E2B2C2E1C1, Q18 Q_Dual_NPN_PNP_B1E2B2C2E1C1, Q19 Q_Dual_NPN_PNP_B1E2B2C2E1C1, Q20 Q_Dual_NPN_PNP_B1E2B2C2E1C1, Q21 Q_Dual_NPN_PNP_B1E2B2C2E1C1, Q22 Q_Dual_NPN_PNP_B1E2B2C2E1C1, Q23 Q_Dual_NPN_PNP_B1E2B2C2E1C1, Q24 Q_Dual_NPN_PNP_B1E2B2C2E1C1, Q25 Q_Dual_NPN_PNP_B1E2B2C2E1C1, Q26 Q_Dual_NPN_PNP_B1E2B2C2E1C1, Q27 Q_Dual_NPN_PNP_B1E2B2C2E1C1, Q28 Q_Dual_NPN_PNP_B1E2B2C2E1C1, Q29 Q_Dual_NPN_PNP_B1E2B2C2E1C1, SW1 SW_Push, SW2 SW_Push, SW3 SW_Push, U1 74AUP1G80, U10 NMUX1308BQ, U11 NMUX1308BQ, U12 NMUX1308BQ, U13 NMUX1308BQ, U14 NMUX1308BQ, U15 NMUX1308BQ, U16 NMUX1308BQ, U17 74AUP1G80, U18 74AHC1G86, U19 74AUP1G80, U20 74AUP1G80, U21 74LV1T08GV, U22 CD74HC283M96, U23 74LV1T08GV, U24 74LVC1GU04DRL, U25 ESP32-S3-MINI-1, U26 74LVC1GU04DRL, U27 74LV1T08GV, U28 CD74HC283M96, U29 NMUX1308BQ, U3 74AHC1G86, U30 NMUX1308BQ, U31 NMUX1308BQ, U32 NMUX1308BQ, U33 74AUP1G80, U34 74AUP1G80, U35 NMUX1308BQ, U36 NMUX1308BQ, U37 74AUP1G80, U38 74AUP1G80, U39 NMUX1308BQ, U4 74AUP1G80, U40 NMUX1308BQ, U41 NMUX1308BQ, U42 NMUX1308BQ, U43 NMUX1308BQ, U44 NMUX1308BQ, U45 74AUP1G80, U46 74AUP1G80, U47 74AUP1G80, U48 74AUP1G80, U49 74AUP1G80, U5 74AUP1G80, U50 74AUP1G80, U51 74LV1T08GV, U52 74AHC1G86, U53 74LVC1GU04DRL, U54 74LVC1GU04DRL, U55 74AHC1G86, U56 74AHC1G86, U57 74LVC1GU04DRL, U58 74LVC1GU04DRL, U59 74LV1T08GV, U6 74AUP1G80, U60 74AHC1G86, U61 74LVC1GU04DRL, U62 74LV1T08GV, U63 74LV1T08GV, U64 NMUX1308BQ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

Commit message: Add files via upload
Add final PCB design
Connections:
- J3 pad SH: (no net) -> Net-(J3-SHIELD)
Routing:
- net Net-(J3-SHIELD): track 15.1 -> 37.4 mm
- net wr3: track 45.3 -> 43.4 mm, vias 4 -> 3
- added copper zone on B.Cu, net GND
- added copper zone on F.Cu, net GND
- added copper zone on In1.Cu, net GND
- added copper zone on In2.Cu, net GND
Changed lines of the file:
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@@
 			(unit
 				(name "A")
-				(pins "B9" "B4" "A4" "A9" "B12" "A1" "A12" "B1" "S1" "A5" "B5" "A7" "B7"
+				(pins "B9" "B4" "A4" "A9" "B12" "A1" "A12" "B1" "SH" "A5" "B5" "A7" "B7"
 					"A6" "B6" "A8" "B8" "A2" "A3" "A10" "A11"
 				)
@@
 			(layers "*.Cu" "*.Mask")
 			(remove_unused_layers no)
+			(net "Net-(J3-SHIELD)")
 		)
 		(pad "SH" thru_hole oval
@@
 			(layers "*.Cu" "*.Mask")
 			(remove_unused_layers no)
+			(net "Net-(J3-SHIELD)")
 		)
 		(pad "SH" thru_hole oval
@@
 			(layers "*.Cu" "*.Mask")
 			(remove_unused_layers no)
+			(net "Net-(J3-SHIELD)")
 		)
 		(pad "SH" thru_hole oval
@@
 			(layers "*.Cu" "*.Mask")
 			(remove_unused_layers no)
+			(net "Net-(J3-SHIELD)")
 		)
 		(embedded_fonts no)
@@
 		(layer "Edge.Cuts")
 	)
+	(point
+		(at 105.15 76.7)
+		(size 1)
+		(layer "B.Cu")
+	)
+	(point
+		(at 105.15 76.7)
+		(size 1)
+		(layer "B.Cu")
+	)
+	(point
+		(at 105.15 76.7)
+		(size 1)
+		(layer "B.Cu")
+	)
+	(point
+		(at 105.15 76.7)
+		(size 1)
+		(layer "B.Cu")
+	)
+	(point
+		(at 105.15 76.7)
+		(size 1)
+		(layer "B.Cu")
+	)
+	(point
+		(at 105.15 76.7)
+		(size 1)
+		(layer "B.Cu")
+	)
+	(point
+		(at 105.15 76.7)
+		(size 1)
+		(layer "B.Cu")
+	)
+	(point
+		(at 105.15 76.7)
+		(size 1)
+		(layer "B.Cu")
+	)
+	(point
+		(at 105.15 76.7)
+		(size 1)
+		(layer "B.Cu")
+	)
+	(point
+		(at 105.15 76.7)
+		(size 1)
+		(layer "B.Cu")
+	)
+	(point
+		(at 105.15 115.5)
+		(size 1)
+		(layer "B.Cu")
+	)
+	(point
+		(at 171.4 76.7)
+		(size 1)
+		(layer "B.Cu")
+	)
+	(point
+		(at 171.4 115.5)
+		(size 1)
+		(layer "B.Cu")
+	)
 	(segment
 		(start 129.598859 80.2)
@@
 	)
 	(segment
+		(start 131.305 84.255)
+		(end 131.305 80.125)
+		(width 0.15)
+		(layer "In1.Cu")
+		(net "Net-(J3-SHIELD)")
+	)
+	(segment
+		(start 131.33 84.28)
+		(end 131.305 84.255)
+		(width 0.15)
+		(layer "In1.Cu")
+		(net "Net-(J3-SHIELD)")
+	)
+	(segment
+		(start 143.39 87.7)
+		(end 143.9 87.7)
+		(width 0.15)
+		(layer "In1.Cu")
+		(net "Net-(J3-SHIELD)")
+	)
+	(segment
+		(start 139.97 80.1)
+		(end 139.97 84.28)
+		(width 0.15)
+		(layer "In1.Cu")
+		(net "Net-(J3-SHIELD)")
+	)
+	(segment
+		(start 131.33 80.1)
+		(end 139.97 80.1)
+		(width 0.15)
+		(layer "In1.Cu")
+		(net "Net-(J3-SHIELD)")
+	)
+	(segment
+		(start 131.305 80.125)
+		(end 131.33 80.1)
+		(width 0.15)
+		(layer "In1.Cu")
+		(net "Net-(J3-SHIELD)")
+	)
+	(segment
+		(start 139.97 84.28)
+		(end 143.39 87.7)
+		(width 0.15)
+		(layer "In1.Cu")
+		(net "Net-(J3-SHIELD)")
+	)
+	(segment
 		(start 142.5 92.25)
 		(end 143.9 90.85)
@@
 		(net "wr3")
 	)
-	(segment
-		(start 161.412782 94.869982)
-		(end 161.412782 95.702181)
-		(width 0.15)
-		(layer "F.Cu")
-		(net "wr3")
-	)
-	(segment
-		(start 161.049981 96.064982)
-		(end 160.537482 96.064982)
-		(width 0.15)
-		(layer "F.Cu")
-		(net "wr3")
-	)
-	(segment
-		(start 161.412782 95.702181)
-		(end 161.049981 96.064982)
-		(width 0.15)
-		(layer "F.Cu")
-		(net "wr3")
-	)
 	(via
 		(at 122.75 100.75)
@@
 	)
 	(via
-		(at 161.412782 94.869982)
-		(size 0.6)
-		(drill 0.3)
-		(layers "F.Cu" "B.Cu")
-		(net "wr3")
-	)
-	(via
 		(at 143.3 98.35)
 		(size 0.6)
@@
 		(net "Net-(U22-A3)")
 	)
+	(zone
+		(net "GND")
+		(layers "F.Cu" "B.Cu" "In1.Cu" "In2.Cu")
+		(hatch edge 0.5)
+		(priority 1)
+		(connect_pads thru_hole_only
+			(clearance 0.12)
+		)
+		(min_thickness 0.15)
+		(fill yes
+			(thermal_gap 0.2)
+			(thermal_bridge_width 0.15)
+			(island_removal_mode 0)
+		)
+		(polygon
+			(pts
+				(xy 105.15 76.7) (xy 105.15 115.5) (xy 171.4 115.5) (xy 171.4 76.7)
+			)
+		)
+	)
+	(zone
+		(net "GND")
+		(layer "B.Cu")
+		(hatch edge 0.5)
+		(connect_pads
+			(clearance 0.12)
+		)
+		(min_thickness 0.15)
+		(fill yes
+			(thermal_gap 0.2)
+			(thermal_bridge_width 0.15)
+			(island_removal_mode 0)
+		)
+		(polygon
+			(pts
+				(xy 105.15 76.7) (xy 105.15 115.5) (xy 171.4 115.5) (xy 171.4 76.7)
+			)
+		)
+	)
 	(embedded_fonts no)
